Commit message: major bug fixing of controller timeout error

File: staubli_tx2_60l_description/urdf/staubli_tx2_60l.urdf.xacro (robot description, xacro)
@@ -7,9 +7,13 @@
         <!--Plunger intervention-->
         <link name="plunger_tooltip"/>
-        <link name="realsense_lidar"/>
+        <link name="camera_color_optical_frame"/>
+        <link name="test"/>
+        <link name="test2"/>
         <!--Petri intervention-->
         <link name="petri_tooltip"/>
-        <link name="petri_pickup"/>
-        <link name="petri_dropoff"/>
+        <!-- <link name="petri_pickup"/>
+        <link name="petri_dropoff"/> -->
+        <!--Stoter intervention-->
+        <link name="stoter_tooltip"/>
         <!--Allignment links-->
         <link name="allignTable"/>
@@ -29,6 +33,16 @@
         <joint name="tool0_to_camera" type="fixed">
             <parent link="tool0"/>
-            <child link="realsense_lidar"/>
+            <child link="camera_color_optical_frame"/>
             <origin xyz="0.0838 0.0845 0.2422" rpy="${radians(-88.6689)} ${radians(0.3632)} ${radians(-44.8563)}"/>
+        </joint>
+        <joint name="base_link_to_test" type="fixed">
+            <parent link="base_link"/>
+            <child link="test"/>
+            <origin xyz="0.7 0.2 0.3" rpy="0 ${radians(180)} 0"/>
+        </joint>
+        <joint name="base_link_to_test2" type="fixed">
+            <parent link="base_link"/>
+            <child link="test2"/>
+            <origin xyz="0.5 -0.2 0.15" rpy="0 ${radians(180)} 0"/>
         </joint>
         <!--Petri intervention-->
@@ -36,7 +50,7 @@
             <parent link="tool0"/>
             <child link="petri_tooltip"/>
-            <origin xyz="0 0 0.290" rpy="0 0 0"/>
+            <origin xyz="0 0 0.2235" rpy="0 0 0"/>
         </joint>
-        <joint name="base_to_petri_pickup" type="fixed">
+        <!-- <joint name="base_to_petri_pickup" type="fixed">
             <parent link="base"/>
             <child link="petri_pickup"/>
@@ -47,4 +61,10 @@
             <child link="petri_dropoff"/>
             <origin xyz ="0.320 0.200 -0.304" rpy="${radians(180)} ${radians(0)} ${radians(0)}"/>
+        </joint> -->
+        <!--Stoter intervention-->
+        <joint name="tool0_to_stoter_tooltip" type="fixed">
+            <parent link="tool0"/>
+            <child link="stoter_tooltip"/>
+            <origin xyz="0.0218 0.0218 0.1355" rpy="${radians(-45)} ${radians(90)} 0"/>
         </joint>
         <!--Allignment joints-->

File: staubli_tx2_60l_moveit_config/config/staubli_tx2_60l.urdf.xacro (robot description, xacro)
@@ -3,5 +3,5 @@
     <xacro:arg name="initial_positions_file" default="initial_positions.yaml" />
     <!-- Import panda urdf file -->
-    <xacro:include filename="$(find staubli_tx2_60l_description)/urdf/staubli_tx2_60l.xacro" />
+    <xacro:include filename="$(find staubli_tx2_60l_description)/urdf/staubli_tx2_60l.urdf.xacro" />
     <!-- Import panda ros2_control description -->
     <xacro:include filename="staubli_tx2_60l.ros2_control.xacro" />

Commit message: Bug fix - correct handling of angular limits

File: staubli_tx2_60l_description/urdf/staubli_tx2_60l.urdf.xacro (robot description, xacro)
@@ -8,10 +8,8 @@
         <link name="plunger_tooltip"/>
         <link name="camera_color_optical_frame"/>
-        <link name="test"/>
-        <link name="test2"/>
         <!--Petri intervention-->
         <link name="petri_tooltip"/>
-        <!-- <link name="petri_pickup"/>
-        <link name="petri_dropoff"/> -->
+        <link name="petri_pickup"/>
+        <link name="petri_dropoff"/>
         <!--Stoter intervention-->
         <link name="stoter_tooltip"/>
@@ -36,14 +34,4 @@
             <origin xyz="0.0838 0.0845 0.2422" rpy="${radians(-88.6689)} ${radians(0.3632)} ${radians(-44.8563)}"/>
         </joint>
-        <joint name="base_link_to_test" type="fixed">
-            <parent link="base_link"/>
-            <child link="test"/>
-            <origin xyz="0.7 0.2 0.3" rpy="0 ${radians(180)} 0"/>
-        </joint>
-        <joint name="base_link_to_test2" type="fixed">
-            <parent link="base_link"/>
-            <child link="test2"/>
-            <origin xyz="0.5 -0.2 0.15" rpy="0 ${radians(180)} 0"/>
-        </joint>
         <!--Petri intervention-->
         <joint name="tool0_to_petri_tooltip" type="fixed">
@@ -52,5 +40,5 @@
             <origin xyz="0 0 0.2235" rpy="0 0 0"/>
         </joint>
-        <!-- <joint name="base_to_petri_pickup" type="fixed">
+        <joint name="base_to_petri_pickup" type="fixed">
             <parent link="base"/>
             <child link="petri_pickup"/>
@@ -61,5 +49,5 @@
             <child link="petri_dropoff"/>
             <origin xyz ="0.320 0.200 -0.304" rpy="${radians(180)} ${radians(0)} ${radians(0)}"/>
-        </joint> -->
+        </joint>
         <!--Stoter intervention-->
         <joint name="tool0_to_stoter_tooltip" type="fixed">
